File: PCB/SakurajimaSplit.kicad_pcb (KiCad board)
At the start: 2 copper layers, 0 parts

Commit message: feat(pcb): add missing 3d models
Parts:
- added C1: 100nF, Capacitor_SMD:C_0603_1608Metric, F.Cu at (-45.1, 107.8)
- added C10: 4.7uF, Capacitor_SMD:C_0805_2012Metric, F.Cu at (-11.0, 111.1)
- added C11: 4.7uF, Capacitor_SMD:C_0805_2012Metric, F.Cu at (-11.0, 114.1)
- added C12: 100nF, Capacitor_SMD:C_0603_1608Metric, F.Cu at (485.4, 156.7)
- added C13: 20pF, Capacitor_SMD:C_0402_1005Metric_Pad0.74x0.62mm_HandSolder, F.Cu at (505.1, 128.4)
- added C14: 20pF, Capacitor_SMD:C_0402_1005Metric_Pad0.74x0.62mm_HandSolder, F.Cu at (505.1, 130.4)
- added C15: 4.7uF, Capacitor_SMD:C_0805_2012Metric, F.Cu at (502.1, 142.8)
- added C16: 100nF, Capacitor_SMD:C_0603_1608Metric, F.Cu at (485.4, 159.2)
- added C17: 100nF, Capacitor_SMD:C_0603_1608Metric, F.Cu at (485.4, 161.7)
- added C18: 100nF, Capacitor_SMD:C_0603_1608Metric, F.Cu at (485.4, 164.2)
- added C19: 100nF, Capacitor_SMD:C_0603_1608Metric, F.Cu at (485.4, 166.7)
- added C2: 20pF, Capacitor_SMD:C_0402_1005Metric_Pad0.74x0.62mm_HandSolder, F.Cu at (-41.1, 134.9)
- added C20: TBD, Capacitor_SMD:C_0805_2012Metric, F.Cu at (440.6, 133.3)
- added C21: 4.7uF, Capacitor_SMD:C_0805_2012Metric, F.Cu at (440.6, 136.3)
- added C22: 4.7uF, Capacitor_SMD:C_0805_2012Metric, F.Cu at (440.6, 139.3)
- added C3: 20pF, Capacitor_SMD:C_0402_1005Metric_Pad0.74x0.62mm_HandSolder, F.Cu at (-41.1, 136.8)
- added C4: 4.7uF, Capacitor_SMD:C_0805_2012Metric, F.Cu at (-44.9, 135.4)
- added C5: 100nF, Capacitor_SMD:C_0603_1608Metric, F.Cu at (-45.1, 110.4)
- added C6: 100nF, Capacitor_SMD:C_0603_1608Metric, F.Cu at (-45.1, 112.9)
- added C7: 100nF, Capacitor_SMD:C_0603_1608Metric, F.Cu at (-45.1, 115.4)
- added C8: 100nF, Capacitor_SMD:C_0603_1608Metric, F.Cu at (-45.1, 117.9)
- added C9: TBD, Capacitor_SMD:C_0805_2012Metric, F.Cu at (-11.0, 108.1)
- added D1: D, Diode_SMD:D_SOD-123, F.Cu at (41.4, 122.7)
- added D10: D, Diode_SMD:D_SOD-123, F.Cu at (98.6, 113.2)
- added D11: D, Diode_SMD:D_SOD-123, F.Cu at (117.6, 118.0)
- added D12: D, Diode_SMD:D_SOD-123, F.Cu at (136.7, 122.7)
- added D13: D, Diode_SMD:D_SOD-123, F.Cu at (41.4, 160.8)
- added D14: D, Diode_SMD:D_SOD-123, F.Cu at (60.5, 160.8)
- added D15: D, Diode_SMD:D_SOD-123, F.Cu at (79.5, 146.5)
- added D16: D, Diode_SMD:D_SOD-123, F.Cu at (98.6, 132.2)
- added D17: D, Diode_SMD:D_SOD-123, F.Cu at (117.6, 137.0)
- added D18: D, Diode_SMD:D_SOD-123, F.Cu at (136.7, 141.8)
- added D19: D, Diode_SMD:D_SOD-123, F.Cu at (141.4, 170.3)
- added D2: D, Diode_SMD:D_SOD-123, F.Cu at (60.5, 122.7)
- added D20: D, Diode_SMD:D_SOD-123, F.Cu at (163.8, 175.7)
- added D21: D, Diode_SMD:D_SOD-123, F.Cu at (180.7, 190.5)
- added D22: D, Diode_SMD:D_SOD-123, F.Cu at (284.3, 103.7)
- added D23: D, Diode_SMD:D_SOD-123, F.Cu at (303.4, 99.3)
- added D24: D, Diode_SMD:D_SOD-123, F.Cu at (322.4, 94.3)
- added D25: D, Diode_SMD:D_SOD-123, F.Cu at (341.5, 108.4)
- added D26: D, Diode_SMD:D_SOD-123, F.Cu at (360.5, 122.7)
- added D27: D, Diode_SMD:D_SOD-123, F.Cu at (379.6, 122.7)
- added D28: D, Diode_SMD:D_SOD-123, F.Cu at (284.3, 122.7)
- added D29: D, Diode_SMD:D_SOD-123, F.Cu at (303.4, 118.0)
- added D3: D, Diode_SMD:D_SOD-123, F.Cu at (79.5, 108.4)
- added D30: D, Diode_SMD:D_SOD-123, F.Cu at (322.4, 113.2)
- added D31: D, Diode_SMD:D_SOD-123, F.Cu at (341.5, 127.5)
- added D32: D, Diode_SMD:D_SOD-123, F.Cu at (360.5, 141.8)
- added D33: D, Diode_SMD:D_SOD-123, F.Cu at (379.6, 141.8)
- added D34: D, Diode_SMD:D_SOD-123, F.Cu at (284.3, 141.8)
- added D35: D, Diode_SMD:D_SOD-123, F.Cu at (303.4, 137.0)
- added D36: D, Diode_SMD:D_SOD-123, F.Cu at (322.4, 132.2)
- added D37: D, Diode_SMD:D_SOD-123, F.Cu at (341.5, 146.5)
- added D38: D, Diode_SMD:D_SOD-123, F.Cu at (360.5, 160.8)
- added D39: D, Diode_SMD:D_SOD-123, F.Cu at (379.6, 160.8)
- added D4: D, Diode_SMD:D_SOD-123, F.Cu at (98.6, 94.1)
- added D40: D, Diode_SMD:D_SOD-123, F.Cu at (240.2, 190.3)
- added D41: D, Diode_SMD:D_SOD-123, F.Cu at (257.2, 175.6)
- added D42: D, Diode_SMD:D_SOD-123, F.Cu at (279.6, 170.3)
- added D43: CapsLock ind., LED_SMD:LED_0603_1608Metric, F.Cu at (-33.1, 107.9)
- added D44: D_Schottky, Diode_SMD:D_SOD-123, F.Cu at (-13.6, 118.3)
- added D45: PWR ind., LED_SMD:LED_0603_1608Metric, F.Cu at (-18.8, 125.1)
- added D46: CapsLock ind., LED_SMD:LED_0603_1608Metric, F.Cu at (485.4, 169.3)
- added D47: D_Schottky, Diode_SMD:D_SOD-123, F.Cu at (445.7, 133.5)
- added D48: PWR ind., LED_SMD:LED_0603_1608Metric, F.Cu at (440.4, 142.1)
- added D5: D, Diode_SMD:D_SOD-123, F.Cu at (117.6, 98.9)
- added D6: D, Diode_SMD:D_SOD-123, F.Cu at (136.7, 103.7)
- added D7: D, Diode_SMD:D_SOD-123, F.Cu at (41.4, 141.8)
- added D8: D, Diode_SMD:D_SOD-123, F.Cu at (60.5, 141.8)
- added D9: D, Diode_SMD:D_SOD-123, F.Cu at (79.5, 127.5)
- added H1: MountingHole, MountingHole:MountingHole_3.2mm_M3_Pad, F.Cu at (-51.1, 110.6)
- added H2: MountingHole, MountingHole:MountingHole_3.2mm_M3_Pad, F.Cu at (-51.1, 118.5)
- added H3: MountingHole, MountingHole:MountingHole_3.2mm_M3_Pad, F.Cu at (-51.1, 126.5)
- added H4: MountingHole, MountingHole:MountingHole_3.2mm_M3_Pad, F.Cu at (-51.1, 134.4)
- added H5: MountingHole, MountingHole:MountingHole_3.2mm_M3_Pad, F.Cu at (487.4, 116.7)
- added H6: MountingHole, MountingHole:MountingHole_3.2mm_M3_Pad, F.Cu at (487.4, 124.6)
- added H7: MountingHole, MountingHole:MountingHole_3.2mm_M3_Pad, F.Cu at (487.4, 132.6)
- added H8: MountingHole, MountingHole:MountingHole_3.2mm_M3_Pad, F.Cu at (487.4, 140.5)
- added J1: SWD, Connector_PinHeader_2.54mm:PinHeader_1x05_P2.54mm_Horizontal, F.Cu at (-52.8, 155.9)
- added J10: Conn_01x01_Pin, Connector_Wire:SolderWirePad_1x01_SMD_1x2mm, F.Cu at (-33.5, 159.1)
- added J11: Conn_01x01_Pin, Connector_Wire:SolderWirePad_1x01_SMD_1x2mm, F.Cu at (-40.5, 162.7)
- added J12: Conn_01x01_Pin, Connector_Wire:SolderWirePad_1x01_SMD_1x2mm, F.Cu at (-38.2, 162.7)
- added J13: Conn_01x01_Pin, Connector_Wire:SolderWirePad_1x01_SMD_1x2mm, F.Cu at (-35.8, 162.7)
- added J14: Conn_01x01_Pin, Connector_Wire:SolderWirePad_1x01_SMD_1x2mm, F.Cu at (-33.5, 162.7)
- added J15: Conn_01x01_Pin, Connector_Wire:SolderWirePad_1x01_SMD_1x2mm, F.Cu at (-40.5, 166.4)
- added J16: Conn_01x01_Pin, Connector_Wire:SolderWirePad_1x01_SMD_1x2mm, F.Cu at (-38.2, 166.4)
- added J17: Conn_01x01_Pin, Connector_Wire:SolderWirePad_1x01_SMD_1x2mm, F.Cu at (-35.8, 166.4)
- added J18: Conn_01x01_Pin, Connector_Wire:SolderWirePad_1x01_SMD_1x2mm, F.Cu at (-33.5, 166.4)
- added J19: USB-C to Host, Connector_USB:USB_C_Receptacle_G-Switch_GT-USB-7010ASV, F.Cu at (-19.0, 112.0)
- added J2: USB-C to Right-Half, Connector_USB:USB_C_Receptacle_G-Switch_GT-USB-7010ASV, F.Cu at (-37.9, 173.8)
- added J20: SWD, Connector_PinHeader_2.54mm:PinHeader_1x05_P2.54mm_Horizontal, F.Cu at (493.6, 115.0)
- added J21: Conn_01x01_Pin, Connector_Wire:SolderWirePad_1x01_SMD_1x2mm, F.Cu at (484.6, 146.3)
- added J22: Conn_01x01_Pin, Connector_Wire:SolderWirePad_1x01_SMD_1x2mm, F.Cu at (486.9, 146.3)
- added J23: Conn_01x01_Pin, Connector_Wire:SolderWirePad_1x01_SMD_1x2mm, F.Cu at (489.3, 146.3)
- added J24: Conn_01x01_Pin, Connector_Wire:SolderWirePad_1x01_SMD_1x2mm, F.Cu at (491.6, 146.3)
- added J25: Conn_01x01_Pin, Connector_Wire:SolderWirePad_1x01_SMD_1x2mm, F.Cu at (494.0, 146.3)
- added J26: Conn_01x01_Pin, Connector_Wire:SolderWirePad_1x01_SMD_1x2mm, F.Cu at (496.4, 146.3)
- added J27: Conn_01x01_Pin, Connector_Wire:SolderWirePad_1x01_SMD_1x2mm, F.Cu at (498.7, 146.3)
- added J28: Conn_01x01_Pin, Connector_Wire:SolderWirePad_1x01_SMD_1x2mm, F.Cu at (484.6, 150.0)
- added J29: Conn_01x01_Pin, Connector_Wire:SolderWirePad_1x01_SMD_1x2mm, F.Cu at (486.9, 150.0)
- added J3: Conn_01x01_Pin, Connector_Wire:SolderWirePad_1x01_SMD_1x2mm, F.Cu at (-40.5, 155.5)
- added J30: Conn_01x01_Pin, Connector_Wire:SolderWirePad_1x01_SMD_1x2mm, F.Cu at (489.3, 150.0)
- added J31: Conn_01x01_Pin, Connector_Wire:SolderWirePad_1x01_SMD_1x2mm, F.Cu at (491.6, 150.0)
- added J32: Conn_01x01_Pin, Connector_Wire:SolderWirePad_1x01_SMD_1x2mm, F.Cu at (494.0, 150.0)
- added J33: Conn_01x01_Pin, Connector_Wire:SolderWirePad_1x01_SMD_1x2mm, F.Cu at (496.4, 150.0)
- added J34: Conn_01x01_Pin, Connector_Wire:SolderWirePad_1x01_SMD_1x2mm, F.Cu at (498.7, 150.0)
- added J35: Conn_01x01_Pin, Connector_Wire:SolderWirePad_1x01_SMD_1x2mm, F.Cu at (484.6, 153.6)
- added J36: Conn_01x01_Pin, Connector_Wire:SolderWirePad_1x01_SMD_1x2mm, F.Cu at (486.9, 153.6)
- added J37: Conn_01x01_Pin, Connector_Wire:SolderWirePad_1x01_SMD_1x2mm, F.Cu at (489.3, 153.6)
- added J38: Conn_01x01_Pin, Connector_Wire:SolderWirePad_1x01_SMD_1x2mm, F.Cu at (491.6, 153.6)
- added J39: USB-C to Right-Half, Connector_USB:USB_C_Receptacle_G-Switch_GT-USB-7010ASV, F.Cu at (444.2, 127.1)
- added J4: Conn_01x01_Pin, Connector_Wire:SolderWirePad_1x01_SMD_1x2mm, F.Cu at (-38.2, 155.5)
- added J5: Conn_01x01_Pin, Connector_Wire:SolderWirePad_1x01_SMD_1x2mm, F.Cu at (-35.8, 155.5)
- added J6: Conn_01x01_Pin, Connector_Wire:SolderWirePad_1x01_SMD_1x2mm, F.Cu at (-33.5, 155.5)
- added J7: Conn_01x01_Pin, Connector_Wire:SolderWirePad_1x01_SMD_1x2mm, F.Cu at (-40.5, 159.1)
- added J8: Conn_01x01_Pin, Connector_Wire:SolderWirePad_1x01_SMD_1x2mm, F.Cu at (-38.2, 159.1)
- added J9: Conn_01x01_Pin, Connector_Wire:SolderWirePad_1x01_SMD_1x2mm, F.Cu at (-35.8, 159.1)
- added JP1: VBUS, Jumper:SolderJumper-2_P1.3mm_Open_TrianglePad1.0x1.5mm, F.Cu at (-18.7, 118.4)
- added JP2: +3.3V, Jumper:SolderJumper-2_P1.3mm_Open_TrianglePad1.0x1.5mm, F.Cu at (-18.7, 122.0)
- added JP3: VBUS, Jumper:SolderJumper-2_P1.3mm_Open_TrianglePad1.0x1.5mm, F.Cu at (436.2, 123.5)
- added JP4: +3.3V, Jumper:SolderJumper-2_P1.3mm_Open_TrianglePad1.0x1.5mm, F.Cu at (436.2, 127.0)
- added JP5: USART_RX, Jumper:SolderJumper-2_P1.3mm_Open_TrianglePad1.0x1.5mm, F.Cu at (436.2, 130.6)
- added JP6: USART_TX, Jumper:SolderJumper-2_P1.3mm_Open_TrianglePad1.0x1.5mm, F.Cu at (436.2, 134.1)
- added L1: 10uH, Inductor_SMD:L_1210_3225Metric, F.Cu at (-13.7, 122.1)
- added L2: 10uH, Inductor_SMD:L_1210_3225Metric, F.Cu at (445.6, 137.2)
- added MX1: SW_Push_45deg, PCM_marbastlib-mx:SW_MX_1u, F.Cu at (41.3, 118.3)
- added MX10: D, PCM_marbastlib-mx:SW_MX_1u, F.Cu at (98.4, 108.7)
- added MX11: F, PCM_marbastlib-mx:SW_MX_1u, F.Cu at (117.5, 113.5)
- added MX12: G, PCM_marbastlib-mx:SW_MX_1u, F.Cu at (136.5, 118.3)
- added MX13: SW_Push_45deg, PCM_marbastlib-mx:SW_MX_1u, F.Cu at (41.3, 156.4)
- added MX14: Z, PCM_marbastlib-mx:SW_MX_1u, F.Cu at (60.3, 156.4)
- added MX15: X, PCM_marbastlib-mx:SW_MX_1u, F.Cu at (79.4, 142.1)
- added MX16: C, PCM_marbastlib-mx:SW_MX_1u, F.Cu at (98.4, 127.8)
- added MX17: V, PCM_marbastlib-mx:SW_MX_1u, F.Cu at (117.5, 132.6)
- added MX18: B, PCM_marbastlib-mx:SW_MX_1u, F.Cu at (136.5, 137.3)
- added MX19: SW_Push_45deg, PCM_marbastlib-mx:SW_MX_1u, F.Cu at (141.3, 165.9)
- added MX2: Q, PCM_marbastlib-mx:SW_MX_1u, F.Cu at (60.3, 118.3)
- added MX20: SW_Push_45deg, PCM_marbastlib-mx:SW_MX_1u, F.Cu at (165.3, 171.5)
- added MX21: SW_Push_45deg, PCM_marbastlib-mx:SW_MX_1u, F.Cu at (183.9, 187.5)
- added MX22: Y, PCM_marbastlib-mx:SW_MX_1u, F.Cu at (284.2, 99.2)
- added MX23: U, PCM_marbastlib-mx:SW_MX_1u, F.Cu at (303.2, 94.8)
- added MX24: I, PCM_marbastlib-mx:SW_MX_1u, F.Cu at (322.3, 89.9)
- added MX25: O, PCM_marbastlib-mx:SW_MX_1u, F.Cu at (341.3, 104.0)
- added MX26: P, PCM_marbastlib-mx:SW_MX_1u, F.Cu at (360.4, 118.3)
- added MX27: SW_Push_45deg, PCM_marbastlib-mx:SW_MX_1u, F.Cu at (379.4, 118.3)
- added MX28: H, PCM_marbastlib-mx:SW_MX_1u, F.Cu at (284.2, 118.3)
- added MX29: J, PCM_marbastlib-mx:SW_MX_1u, F.Cu at (303.2, 113.5)
- added MX3: W, PCM_marbastlib-mx:SW_MX_1u, F.Cu at (79.4, 104.0)
- added MX30: K, PCM_marbastlib-mx:SW_MX_1u, F.Cu at (322.3, 108.7)
- added MX31: L, PCM_marbastlib-mx:SW_MX_1u, F.Cu at (341.3, 123.0)
- added MX32: ; :, PCM_marbastlib-mx:SW_MX_1u, F.Cu at (360.4, 137.3)
- added MX33: ' ", PCM_marbastlib-mx:SW_MX_1u, F.Cu at (379.4, 137.3)
- added MX34: N, PCM_marbastlib-mx:SW_MX_1u, F.Cu at (284.2, 137.3)
- added MX35: M, PCM_marbastlib-mx:SW_MX_1u, F.Cu at (303.2, 132.6)
- added MX36: , <, PCM_marbastlib-mx:SW_MX_1u, F.Cu at (322.3, 127.8)
- added MX37: . >, PCM_marbastlib-mx:SW_MX_1u, F.Cu at (341.3, 142.1)
- added MX38: / ?, PCM_marbastlib-mx:SW_MX_1u, F.Cu at (360.4, 156.4)
- added MX39: SW_Push_45deg, PCM_marbastlib-mx:SW_MX_1u, F.Cu at (379.4, 156.4)
- added MX4: E, PCM_marbastlib-mx:SW_MX_1u, F.Cu at (98.4, 89.7)
- added MX40: SW_Push_45deg, PCM_marbastlib-mx:SW_MX_1u, F.Cu at (236.7, 187.5)
- added MX41: SW_Push_45deg, PCM_marbastlib-mx:SW_MX_1u, F.Cu at (255.4, 171.5)
- added MX42: SW_Push_45deg, PCM_marbastlib-mx:SW_MX_1u, F.Cu at (279.4, 165.9)
- added MX5: R, PCM_marbastlib-mx:SW_MX_1u, F.Cu at (117.5, 94.5)
- added MX6: T, PCM_marbastlib-mx:SW_MX_1u, F.Cu at (136.5, 99.2)
- added MX7: SW_Push_45deg, PCM_marbastlib-mx:SW_MX_1u, F.Cu at (41.3, 137.3)
- added MX8: A, PCM_marbastlib-mx:SW_MX_1u, F.Cu at (60.3, 137.3)
- added MX9: S, PCM_marbastlib-mx:SW_MX_1u, F.Cu at (79.4, 123.0)
- added R1: 330R, Resistor_SMD:R_0603_1608Metric, F.Cu at (-41.1, 107.8)
- added R10: 5.1k, Resistor_SMD:R_0603_1608Metric, F.Cu at (-22.9, 120.4)
- added R11: 330R, Resistor_SMD:R_0603_1608Metric, F.Cu at (-22.9, 122.9)
- added R12: 330R, Resistor_SMD:R_0603_1608Metric, F.Cu at (489.4, 156.7)
- added R13: TBD, Resistor_SMD:R_0603_1608Metric, F.Cu at (489.4, 159.2)
- added R14: 10k, Resistor_SMD:R_0603_1608Metric, F.Cu at (489.4, 161.7)
- added R15: 10k, Resistor_SMD:R_0603_1608Metric, F.Cu at (489.4, 164.2)
- added R16: 10k, Resistor_SMD:R_0603_1608Metric, F.Cu at (489.4, 166.7)
- added R17: 10k, Resistor_SMD:R_0603_1608Metric, F.Cu at (493.4, 156.7)
- added R18: 10k, Resistor_SMD:R_0603_1608Metric, F.Cu at (493.4, 159.2)
- added R19: 10k, Resistor_SMD:R_0603_1608Metric, F.Cu at (493.4, 161.7)
- added R2: TBD, Resistor_SMD:R_0603_1608Metric, F.Cu at (-41.1, 110.4)
- added R20: 330R, Resistor_SMD:R_0603_1608Metric, F.Cu at (436.0, 137.2)
- added R3: 10k, Resistor_SMD:R_0603_1608Metric, F.Cu at (-41.1, 112.9)
- added R4: 10k, Resistor_SMD:R_0603_1608Metric, F.Cu at (-41.1, 115.4)
- added R5: 10k, Resistor_SMD:R_0603_1608Metric, F.Cu at (-41.1, 117.9)
- added R6: 10k, Resistor_SMD:R_0603_1608Metric, F.Cu at (-37.1, 107.8)
- added R7: 10k, Resistor_SMD:R_0603_1608Metric, F.Cu at (-37.1, 110.4)
- added R8: 10k, Resistor_SMD:R_0603_1608Metric, F.Cu at (-37.1, 112.9)
- added R9: 5.1k, Resistor_SMD:R_0603_1608Metric, F.Cu at (-22.9, 117.9)
- added SW1: SWCLK/BOOT0, Button_Switch_SMD:SW_Push_1P1T_XKB_TS-1187A, F.Cu at (-42.9, 130.6)
- added SW2: Knob, Rotary_Encoder:RotaryEncoder_Alps_EC11E-Switch_Vertical_H20mm, F.Cu at (-80.7, 109.3)
- added SW3: SWCLK/BOOT0, Button_Switch_SMD:SW_Push_1P1T_XKB_TS-1187A, F.Cu at (495.6, 138.9)
- added SW4: Knob, Rotary_Encoder:RotaryEncoder_Alps_EC11E-Switch_Vertical_H20mm, F.Cu at (485.4, 102.6)
- added TP1: USART_TX, TestPoint:TestPoint_Pad_2.0x2.0mm, F.Cu at (-45.1, 121.2)
- added TP10: +5V, TestPoint:TestPoint_Pad_2.0x2.0mm, F.Cu at (-26.9, 112.7)
- added TP11: +3.3V, TestPoint:TestPoint_Pad_2.0x2.0mm, F.Cu at (-26.9, 116.7)
- added TP12: USB_D-, TestPoint:TestPoint_Pad_2.0x2.0mm, F.Cu at (-26.9, 120.8)
- added TP13: USB_D+, TestPoint:TestPoint_Pad_2.0x2.0mm, F.Cu at (-26.9, 124.8)
- added TP14: GND, TestPoint:TestPoint_Pad_2.0x2.0mm, F.Cu at (493.4, 129.5)
- added TP15: GND, TestPoint:TestPoint_Pad_2.0x2.0mm, F.Cu at (493.4, 133.5)
- added TP16: GND, TestPoint:TestPoint_Pad_2.0x2.0mm, F.Cu at (497.4, 129.5)
- added TP17: GND, TestPoint:TestPoint_Pad_2.0x2.0mm, F.Cu at (497.4, 133.5)
- added TP18: Display_SCLK, TestPoint:TestPoint_Pad_2.0x2.0mm, F.Cu at (501.5, 129.5)
- added TP19: Display_SDI, TestPoint:TestPoint_Pad_2.0x2.0mm, F.Cu at (501.5, 133.5)
- added TP2: USART_RX, TestPoint:TestPoint_Pad_2.0x2.0mm, F.Cu at (-45.1, 125.2)
- added TP20: VBUS, TestPoint:TestPoint_Pad_2.0x2.0mm, F.Cu at (432.0, 123.7)
- added TP21: +5V, TestPoint:TestPoint_Pad_2.0x2.0mm, F.Cu at (432.0, 127.8)
- added TP22: +3.3V, TestPoint:TestPoint_Pad_2.0x2.0mm, F.Cu at (432.0, 131.8)
- added TP23: USART_RX, TestPoint:TestPoint_Pad_2.0x2.0mm, F.Cu at (432.0, 135.9)
- added TP24: USART_TX, TestPoint:TestPoint_Pad_2.0x2.0mm, F.Cu at (432.0, 139.9)
- added TP3: GND, TestPoint:TestPoint_Pad_2.0x2.0mm, F.Cu at (-41.1, 121.2)
- added TP4: GND, TestPoint:TestPoint_Pad_2.0x2.0mm, F.Cu at (-41.1, 125.2)
- added TP5: GND, TestPoint:TestPoint_Pad_2.0x2.0mm, F.Cu at (-37.0, 121.2)
- added TP6: GND, TestPoint:TestPoint_Pad_2.0x2.0mm, F.Cu at (-37.0, 125.2)
- added TP7: Display_SCLK, TestPoint:TestPoint_Pad_2.0x2.0mm, F.Cu at (-33.0, 121.2)
- added TP8: Display_SDI, TestPoint:TestPoint_Pad_2.0x2.0mm, F.Cu at (-33.0, 125.2)
- added TP9: VBUS, TestPoint:TestPoint_Pad_2.0x2.0mm, F.Cu at (-26.9, 108.6)
- added U1: USBLC6-2SC6, Package_TO_SOT_SMD:SOT-23-6, F.Cu at (-36.0, 135.4)
- added U2: STM32G0B1CBT6, Package_QFP:LQFP-48_7x7mm_P0.5mm, F.Cu at (-49.4, 174.1)
- added U3: ZJY_M233, Hayata_Lib:OLED_SSD1305, F.Cu at (-68.3, 143.7)
- added U4: TLV76733DRVR, Package_SON:WSON-6-1EP_2x2mm_P0.65mm_EP1x1.6mm_ThermalVias, F.Cu at (-22.8, 126.1)
- added U5: USBLC6-2SC6, Package_TO_SOT_SMD:SOT-23-6, F.Cu at (-14.0, 126.6)
- added U6: STM32G0B1CBT6, Package_QFP:LQFP-48_7x7mm_P0.5mm, F.Cu at (501.1, 161.1)
- added U7: ZJY_M233, Hayata_Lib:OLED_SSD1305, F.Cu at (470.2, 134.5)
- added U8: TLV76733DRVR, Package_SON:WSON-6-1EP_2x2mm_P0.65mm_EP1x1.6mm_ThermalVias, F.Cu at (436.1, 140.3)
- added U9: USBLC6-2SC6, Package_TO_SOT_SMD:SOT-23-6, F.Cu at (445.4, 141.7)
- added Y1: 8MHz, Crystal:Crystal_SMD_3225-4Pin_3.2x2.5mm_HandSoldering, F.Cu at (-35.3, 130.1)
- added Y2: 8MHz, Crystal:Crystal_SMD_3225-4Pin_3.2x2.5mm_HandSoldering, F.Cu at (503.2, 138.4)
