File: PCB/SakurajimaSplit.kicad_pcb (KiCad board)
At the start: 2 copper layers, 302 x 112 mm, 192 parts, among them J1 SWD, J2 USB-C to Right-Half, J3 VREF+, J4 SWD, J5 USB-C to Host, J6 VREF+, J7 USB-C to Left-Half, SW1 SWCLK/BOOT0, SW2 SWCLK/BOOT0, U1 USBLC6-2SC6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

Commit message: feat(pcb): add stitching vias
Parts:
- moved C2 22.7 mm to (194.4, 139.9)
- moved J1 22.7 mm to (172.2, 108.3)
- moved JP1 22.7 mm to (180.9, 109.4)
- moved L1 22.7 mm to (177.7, 113.1)
- moved MX11 22.7 mm to (148.1, 130.7)
- moved MX17 22.7 mm to (148.1, 149.7)
- moved MX5 22.7 mm to (148.1, 111.6)
- moved R4 22.7 mm to (194.8, 112.7)
- moved R9 22.7 mm to (196.8, 105.3)
- moved SW1 22.7 mm to (198.6, 146.4)
- moved TP1 22.7 mm to (188.9, 150.5)
- moved TP13 22.7 mm to (187.5, 112.7)
- moved TP2 22.7 mm to (191.3, 150.5)
- moved TP4 22.7 mm to (198.8, 121.3)
- moved TP6 22.7 mm to (196.4, 121.3)
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Routing:
- net GND: track 10.8 -> 7.85 mm, vias 3 -> 214
Other:
- board size 302 x 112 mm -> 300 x 126.4 mm
